File: Design-files/Main/power.kicad_sch (KiCad schematic)
At the start: 15 parts, among them J2 Conn_01x02_Pin, U3 HT75xx-1-SOT89, U4 LTC4054ES5-4.2, U6 TPS2115A-Q1

Commit message: Lots of changes :)
Parts:
- removed U3: HT75xx-1-SOT89, Package_TO_SOT_SMD:SOT-89-3, symbol Regulator_Linear:HT75xx-1-SOT89
- added C5, C6: 1 uF, Capacitor_SMD:C_0201_0603Metric, symbol Device:C
- added J10: BIPP Connection, symbol Connector:Conn_01x01_Pin
- added J11: Switched Power Pin, symbol Connector:Conn_01x01_Pin
- added J8: 3v3 Backup Pin, symbol Connector:Conn_01x01_Pin
- added J8: USB 5V, symbol Connector:Conn_01x01_Pin
- added U7: RT9073A, symbol Power_Management:RT9701
- BT1: footprint (none) -> Battery:BatteryHolder_Keystone_1042_1x18650
- C1, C2, C3, C4: footprint (none) -> Capacitor_SMD:C_0201_0603Metric
- ChargingStatusLED1: footprint (none) -> LED_SMD:LED_0805_2012Metric
- D1: footprint (none) -> Diode_SMD:D_SMA
- J2: value Conn_01x02_Pin -> Battery Jumper; footprint (none) -> Connector_PinHeader_2.54mm:PinHeader_1x02_P2.54mm_Vertical
- R1, R4, R5, Rprog1: footprint (none) -> Resistor_SMD:R_0201_0603Metric
- U6: footprint (none) -> Package_TO_SOT_SMD:TSOT-23-8
Connections:
- net Battery Input Polarity Protection: now also J10.1 (Pin_1)
- net GND: now also C5.2, C6.2, U7.2 (GND)
- net Regulated 3v3: now also C6.1, U7.1 (VOUT), U7.5 (VOUT)
- net Switched Power: now also C5.1, J11.1 (Pin_1), U7.3 (VIN), U7.4 (VIN/EN)
- net USB 5V: now also J8.1 (Pin_1)
- new net 3v3 Regulated: J8.1 (Pin_1)
- no-connect marks 0 -> 1
Other:
- note added: "Regulated Voltage With UVLO"
- note added: "These pins are in case of failure/ incorrect design. By plugging in a new circuit to whatever pins are required would allow for modules to be replaced."
- note removed: "Regulated Voltage"
