File: Design-files/Main/power.kicad_sch (KiCad schematic)
At the start: 24 parts, among them J2 Battery Jumper, J8 Conn_01x04_Pin, U4 LTC4054ES5-4.2, U6 TPS2115A-Q1, U7 RT9073A

Commit message: changes
Parts:
- J8: footprint (none) -> Connector_PinHeader_2.54mm:PinHeader_1x04_P2.54mm_Vertical
- R10, R16, R6, R7, R8, R9: footprint (none) -> Resistor_SMD:R_0201_0603Metric
- Rprog1: value 2000 -> 1000
- U7: footprint (none) -> REG_RT9080-33GQZ:REG_RT9080-33GQZ
Changed lines of the file:
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@@
       (effects (font (size 1.27 1.27)))
     )
-    (property "Footprint" "" (at 149.225 60.198 90)
+    (property "Footprint" "Resistor_SMD:R_0201_0603Metric" (at 149.225 60.198 90)
       (effects (font (size 1.27 1.27)) hide)
     )
@@
       (effects (font (size 1.27 1.27)))
     )
-    (property "Footprint" "" (at 47.752 166.37 90)
+    (property "Footprint" "Resistor_SMD:R_0201_0603Metric" (at 47.752 166.37 90)
       (effects (font (size 1.27 1.27)) hide)
     )
@@
       (effects (font (size 1.27 1.27)))
     )
-    (property "Footprint" "" (at 60.325 104.14 0)
+    (property "Footprint" "REG_RT9080-33GQZ:REG_RT9080-33GQZ" (at 60.325 104.14 0)
       (effects (font (size 1.27 1.27)) hide)
     )
@@
       (effects (font (size 1.27 1.27)) (justify left))
     )
-    (property "Value" "2000" (at 68.58 146.685 0)
+    (property "Value" "1000" (at 68.58 146.685 0)
       (effects (font (size 1.27 1.27)) (justify left))
     )
@@
       (effects (font (size 1.27 1.27)))
     )
-    (property "Footprint" "" (at 78.867 95.885 90)
+    (property "Footprint" "Resistor_SMD:R_0201_0603Metric" (at 78.867 95.885 90)
       (effects (font (size 1.27 1.27)) hide)
     )
@@
       (effects (font (size 1.27 1.27)))
     )
-    (property "Footprint" "" (at 148.59 56.388 90)
+    (property "Footprint" "Resistor_SMD:R_0201_0603Metric" (at 148.59 56.388 90)
       (effects (font (size 1.27 1.27)) hide)
     )
@@
       (effects (font (size 1.27 1.27)))
     )
-    (property "Footprint" "" (at 33.655 154.178 90)
+    (property "Footprint" "Resistor_SMD:R_0201_0603Metric" (at 33.655 154.178 90)
       (effects (font (size 1.27 1.27)) hide)
     )
@@
       (effects (font (size 1.27 1.27)))
     )
-    (property "Footprint" "" (at 59.69 46.863 90)
+    (property "Footprint" "Resistor_SMD:R_0201_0603Metric" (at 59.69 46.863 90)
       (effects (font (size 1.27 1.27)) hide)
     )
@@
       (effects (font (size 1.27 1.27)))
     )
-    (property "Footprint" "" (at 115.57 108.585 0)
-      (effects (font (size 1.27 1.27)) hide)
-    )
+    (property "Footprint" "Connector_PinHeader_2.54mm:PinHeader_1x04_P2.54mm_Vertical" (at 115.57 108.585 0)
+      (effects (font (size 1.27 1.27)) hide)
+    )

Commit message: lets go team
Parts:
- R1, Rprog1: value 1000 -> 1k
Other:
- note added: "Jumper will be placed here to connect these pins. This is incase the battery module is not used"
- moved on the sheet: C2, ChargingStatusLED1, R1, R10, R16, Rprog1, U4

Commit message: lots of changes
Parts:
- removed C5, C6: 1 uF, Capacitor_SMD:C_0201_0603Metric, symbol Device:C
- removed R9: 0, Resistor_SMD:R_0201_0603Metric, symbol Device:R
- removed U6: TPS2115A-Q1, Package_TO_SOT_SMD:TSOT-23-8, symbol Custom:TPS2115A-Q1
- removed U7: RT9073A, REG_RT9080-33GQZ:REG_RT9080-33GQZ, symbol Power_Management:RT9701
- added C10, C11: 1 uF, footprint:C0402, symbol Device:C
- added R28: 0, footprint:R0402, symbol Device:R
- added U5: RT9073A-33GQZ, footprint:ZQFN-4L_L1.0-W1.0-P0.63-BL-EP, symbol RT9073A-33GQZ:RT9073A-33GQZ
- added U6: TPS2115ADRBR, footprint:SON-8_L3.0-W3.0-P0.65-LS3.0-BL-EP, symbol TPS2115ADRBR:TPS2115ADRBR
- C1: footprint Capacitor_SMD:C_0201_0603Metric -> footprint:C0603
- C2: footprint Capacitor_SMD:C_0201_0603Metric -> footprint:C0402
- C3, C4: footprint Capacitor_SMD:C_0201_0603Metric -> footprint:C1206
- ChargingStatusLED1: footprint LED_SMD:LED_0805_2012Metric -> footprint:LED0805-RD
- D1: footprint Diode_SMD:D_SMA -> footprint:SMA_L4.2-W2.6-LS5.3-RD
- R1, Rprog1: footprint Resistor_SMD:R_0201_0603Metric -> footprint:R1206
- R10, R16, R6, R7, R8: footprint Resistor_SMD:R_0201_0603Metric -> footprint:R0402
- R4: value 10K -> 700; footprint Resistor_SMD:R_0201_0603Metric -> footprint:R0603
- R5: value 700 -> 10K; footprint Resistor_SMD:R_0201_0603Metric -> footprint:R0805
Connections:
- net Battery Input Polarity Protection: now also U6.6 (IN2)
- net GND: now also R4.2, C11.2, U5.2 (GND), U6.5 (GND), U6.9 (GND); no longer R4.1, R5.2
- net Regulated 3v3: now also R28.1
- net Switched Power: now also R8.2; no longer R7.2
- net USB 5V: now also R7.2; no longer R8.2
- net at R7.1: now also C4.2, U6.8 (IN1); no longer R4.2
- net at R8.1: now also R5.2, U6.7 (OUT); no longer C4.2
- net at R5.1: now also U6.1 (STAT)
- new net: C11.1, R28.2, U5.1 (VOUT)
- new net: R4.1, U6.4 (ILIM)
- new net: C10.1, U5.3 (EN), U5.5 (SGND)
- new net: C10.2, U5.4 (VIN)
- no-connect marks 1 -> 2
Other:
- note removed: "Regulated Voltage With UVLO"

Commit message: fixed shematic
Parts:
- removed C10: 1 uF, footprint:C0402, symbol Device:C
- added C8: 1 uF, footprint:C0402, symbol Device:C
Connections:
- net GND: now also U5.5 (SGND), C8.2
- net Switched Power: now also U5.3 (EN), U5.4 (VIN), C8.1
Changed lines of the file:
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@@
   (junction (at 104.775 66.04) (diameter 0) (color 0 0 0 0)
   )
-  (junction (at 48.895 99.06) (diameter 0) (color 0 0 0 0)
-  )
   (junction (at 79.375 116.205) (diameter 0) (color 0 0 0 0)
   )
   (junction (at 137.16 58.42) (diameter 0) (color 0 0 0 0)
+  )
+  (junction (at 40.64 106.68) (diameter 0) (color 0 0 0 0)
+  )
+  (junction (at 45.085 106.68) (diameter 0) (color 0 0 0 0)
   )
   (junction (at 140.97 63.5) (diameter 0) (color 0 0 0 0)
@@
     (stroke (width 0) (type default))
   )
+  (wire (pts (xy 34.29 92.075) (xy 34.29 106.68))
+    (stroke (width 0) (type default))
+  )
   (wire (pts (xy 45.72 45.085) (xy 45.72 48.895))
     (stroke (width 0) (type default))
@@
     (stroke (width 0) (type default))
   )
+  (wire (pts (xy 34.29 106.68) (xy 40.64 106.68))
+    (stroke (width 0) (type default))
+  )
   (wire (pts (xy 153.67 58.42) (xy 161.925 58.42))
     (stroke (width 0) (type default))
@@
     (stroke (width 0) (type default))
   )
+  (wire (pts (xy 45.085 106.68) (xy 51.435 106.68))
+    (stroke (width 0) (type default))
+  )
   (wire (pts (xy 120.65 111.125) (xy 134.62 111.125))
     (stroke (width 0) (type default))
@@
     (stroke (width 0) (type default))
   )
-  (wire (pts (xy 48.895 99.06) (xy 51.435 99.06))
-    (stroke (width 0) (type default))
-  )
   (wire (pts (xy 79.375 93.98) (xy 79.375 95.885))
     (stroke (width 0) (type default))
@@
     (stroke (width 0) (type default))
   )
+  (wire (pts (xy 45.085 99.06) (xy 45.085 106.68))
+    (stroke (width 0) (type default))
+  )
   (wire (pts (xy 83.185 98.425) (xy 83.185 95.885))
     (stroke (width 0) (type default))
@@
     (stroke (width 0) (type default))
   )
-  (wire (pts (xy 40.64 99.06) (xy 48.895 99.06))
-    (stroke (width 0) (type default))
-  )
   (wire (pts (xy 130.175 55.88) (xy 131.445 55.88))
     (stroke (width 0) (type default))
   )
+  (wire (pts (xy 45.085 99.06) (xy 51.435 99.06))
+    (stroke (width 0) (type default))
+  )
   (wire (pts (xy 140.97 71.12) (xy 140.97 74.295))
     (stroke (width 0) (type default))
@@
     (stroke (width 0) (type default))
   )
-  (wire (pts (xy 40.64 106.68) (xy 51.435 106.68))
+  (wire (pts (xy 34.925 92.075) (xy 34.29 92.075))
     (stroke (width 0) (type default))
   )
@@
     (stroke (width 0) (type default))
   )
+  (wire (pts (xy 40.64 106.68) (xy 45.085 106.68))
+    (stroke (width 0) (type default))
+  )
   (wire (pts (xy 130.175 63.5) (xy 137.795 63.5))
     (stroke (width 0) (type default))
   )
   (wire (pts (xy 102.235 66.04) (xy 104.775 66.04))
-    (stroke (width 0) (type default))
-  )
-  (wire (pts (xy 48.895 93.345) (xy 48.895 99.06))
     (stroke (width 0) (type default))
   )
@@
   )
   (label "Battery Input Polarity Protection" (at 59.69 36.195 0) (fields_autoplaced)
+    (effects (font (size 1.27 1.27)) (justify left bottom))
+  )
+  (label "Switched Power" (at 34.925 92.075 0) (fields_autoplaced)
     (effects (font (size 1.27 1.27)) (justify left bottom))
   )
@@
     )
   )
+  (symbol (lib_id "power:GND") (at 48.895 93.345 0) (unit 1)
+    (in_bom yes) (on_board yes) (dnp no) (fields_autoplaced)
+    (property "Reference" "#PWR019" (at 48.895 99.695 0)
+      (effects (font (size 1.27 1.27)) hide)
+    )
+    (property "Value" "GND" (at 48.895 99.0385 0)
+      (effects (font (size 1.27 1.27)))
+    )
+    (property "Footprint" "" (at 48.895 93.345 0)
+      (effects (font (size 1.27 1.27)) hide)
+    )
+    (property "Datasheet" "" (at 48.895 93.345 0)
+      (effects (font (size 1.27 1.27)) hide)
+    )
+    (pin "1")
+    (instances
+      (project "Main"
+        (path "/1e9f3d34-a4c0-4684-8b0d-9d61663dabf9/68b97cb2-585c-4237-bacc-43c945d9635d"
+          (reference "#PWR019") (unit 1)
+        )
+      )
+    )
+  )
   (symbol (lib_id "Device:R") (at 210.185 69.85 0) (unit 1)
     (in_bom yes) (on_board yes) (dnp no)
@@
         (path "/1e9f3d34-a4c0-4684-8b0d-9d61663dabf9/68b97cb2-585c-4237-bacc-43c945d9635d"
           (reference "C11") (unit 1)
+        )
+      )
+    )
+  )
+  (symbol (lib_id "Device:C") (at 40.64 110.49 0) (unit 1)
+    (in_bom yes) (on_board yes) (dnp no) (fields_autoplaced)
+    (property "Reference" "C8" (at 44.45 109.855 0)
+      (effects (font (size 1.27 1.27)) (justify left))
+    )
+    (property "Value" "1 uF" (at 44.45 112.395 0)
+      (effects (font (size 1.27 1.27)) (justify left))
+    )
+    (property "Footprint" "footprint:C0402" (at 41.6052 114.3 0)
+      (effects (font (size 1.27 1.27)) hide)
+    )
+    (property "Datasheet" "~" (at 40.64 110.49 0)
+      (effects (font (size 1.27 1.27)) hide)
+    )
+    (pin "1")
+    (pin "2")
+    (instances
+      (project "Main"
+        (path "/1e9f3d34-a4c0-4684-8b0d-9d61663dabf9/68b97cb2-585c-4237-bacc-43c945d9635d"
+          (reference "C8") (unit 1)
         )
       )
@@
     )
   )
+  (symbol (lib_id "power:GND") (at 40.64 114.3 0) (unit 1)
+    (in_bom yes) (on_board yes) (dnp no) (fields_autoplaced)
+    (property "Reference" "#PWR021" (at 40.64 120.65 0)
+      (effects (font (size 1.27 1.27)) hide)
+    )
+    (property "Value" "GND" (at 40.64 119.9935 0)
+      (effects (font (size 1.27 1.27)))
+    )
+    (property "Footprint" "" (at 40.64 114.3 0)
+      (effects (font (size 1.27 1.27)) hide)
+    )
+    (property "Datasheet" "" (at 40.64 114.3 0)
+      (effects (font (size 1.27 1.27)) hide)
+    )
+    (pin "1")
+    (instances
+      (project "Main"
+        (path "/1e9f3d34-a4c0-4684-8b0d-9d61663dabf9/68b97cb2-585c-4237-bacc-43c945d9635d"
+          (reference "#PWR021") (unit 1)
+        )
+      )
+    )
+  )
   (symbol (lib_id "Battery_Management:LTC4054ES5-4.2") (at 210.185 55.88 180) (unit 1)
     (in_bom yes) (on_board yes) (dnp no)
@@
         )
       )
-    )
-  )
-  (symbol (lib_id "Device:C") (at 40.64 102.87 0) (unit 1)
-    (in_bom yes) (on_board yes) (dnp no) (fields_autoplaced)
-    (property "Reference" "C10" (at 44.45 102.235 0)
-      (effects (font (size 1.27 1.27)) (justify left))
-    )
-    (property "Value" "1 uF" (at 44.45 104.775 0)
-      (effects (font (size 1.27 1.27)) (justify left))
-    )
-    (property "Footprint" "footprint:C0402" (at 41.6052 106.68 0)
-      (effects (font (size 1.27 1.27)) hide)
-    )
-    (property "Datasheet" "~" (at 40.64 102.87 0)
-      (effects (font (size 1.27 1.27)) hide)
-    )
-    (pin "1")
-    (pin "2")
-    (instances
-      (project "Main"
-        (path "/1e9f3d34-a4c0-4684-8b0d-9d61663dabf9/68b97cb2-585c-4237-bacc-43c945d9635d"
-          (reference "C10") (unit 1)
-        )
-      )
