File: Design-files/Main/Main.kicad_sch (KiCad schematic)
At the start: 0 parts

Commit message: Lots of changes :)
Other:
- sheet Interfacing ports: added none; removed AnalogueSensorOut
- sheet Sensing Module ports: added none; removed AnalogueSensorOut
Changed lines of the file:
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@@
 (kicad_sch (version 20230121) (generator eeschema)
   (paper "A4")
-  (global_label "Regulated 3v3" (shape input) (at 88.265 137.16 0) (fields_autoplaced)
-    (effects (font (size 1.27 1.27)) (justify left))
-    (property "Intersheetrefs" "${INTERSHEET_REFS}" (at 104.7535 137.16 0)
-      (effects (font (size 1.27 1.27)) (justify left) hide)
-    )
+  (label "DigitalSensorSCL" (at 88.265 146.685 0) (fields_autoplaced)
+    (effects (font (size 1.27 1.27)) (justify left bottom))
   )
-  (global_label "DigitalSensorSCL" (shape input) (at 219.075 62.865 180) (fields_autoplaced)
-    (effects (font (size 1.27 1.27)) (justify right))
-    (property "Intersheetrefs" "${INTERSHEET_REFS}" (at 200.0827 62.865 0)
-      (effects (font (size 1.27 1.27)) (justify right) hide)
-    )
+  (label "Regulated 3v3" (at 219.075 38.1 180) (fields_autoplaced)
+    (effects (font (size 1.27 1.27)) (justify right bottom))
   )
-  (global_label "Regulated 3v3" (shape input) (at 219.075 38.1 180) (fields_autoplaced)
-    (effects (font (size 1.27 1.27)) (justify right))
-    (property "Intersheetrefs" "${INTERSHEET_REFS}" (at 202.5865 38.1 0)
-      (effects (font (size 1.27 1.27)) (justify right) hide)
-    )
+  (label "Regulated 3v3" (at 88.265 137.16 0) (fields_autoplaced)
+    (effects (font (size 1.27 1.27)) (justify left bottom))
   )
-  (global_label "Regulated 3v3" (shape input) (at 87.63 50.8 0) (fields_autoplaced)
-    (effects (font (size 1.27 1.27)) (justify left))
-    (property "Intersheetrefs" "${INTERSHEET_REFS}" (at 104.1185 50.8 0)
-      (effects (font (size 1.27 1.27)) (justify left) hide)
-    )
+  (label "Regulated 3v3" (at 87.63 50.8 0) (fields_autoplaced)
+    (effects (font (size 1.27 1.27)) (justify left bottom))
   )
-  (global_label "DigitalSensorSCL" (shape input) (at 88.265 146.685 0) (fields_autoplaced)
-    (effects (font (size 1.27 1.27)) (justify left))
-    (property "Intersheetrefs" "${INTERSHEET_REFS}" (at 107.2573 146.685 0)
-      (effects (font (size 1.27 1.27)) (justify left) hide)
-    )
+  (label "USB 5V" (at 219.075 24.765 180) (fields_autoplaced)
+    (effects (font (size 1.27 1.27)) (justify right bottom))
   )
-  (global_label "AnalogueSensorOut" (shape input) (at 219.075 76.2 180) (fields_autoplaced)
-    (effects (font (size 1.27 1.27)) (justify right))
-    (property "Intersheetrefs" "${INTERSHEET_REFS}" (at 197.9662 76.2 0)
-      (effects (font (size 1.27 1.27)) (justify right) hide)
-    )
+  (label "DigitalSensorSDA" (at 219.075 67.31 180) (fields_autoplaced)
+    (effects (font (size 1.27 1.27)) (justify right bottom))
   )
-  (global_label "USB 5V" (shape input) (at 219.075 24.765 180) (fields_autoplaced)
-    (effects (font (size 1.27 1.27)) (justify right))
-    (property "Intersheetrefs" "${INTERSHEET_REFS}" (at 209.2991 24.765 0)
-      (effects (font (size 1.27 1.27)) (justify right) hide)
-    )
+  (label "USB 5V" (at 87.63 43.18 0) (fields_autoplaced)
+    (effects (font (size 1.27 1.27)) (justify left bottom))
   )
-  (global_label "DigitalSensorSDA" (shape input) (at 219.075 67.31 180) (fields_autoplaced)
-    (effects (font (size 1.27 1.27)) (justify right))
-    (property "Intersheetrefs" "${INTERSHEET_REFS}" (at 200.0222 67.31 0)
-      (effects (font (size 1.27 1.27)) (justify right) hide)
-    )
+  (label "DigitalSensorSCL" (at 219.075 62.865 180) (fields_autoplaced)
+    (effects (font (size 1.27 1.27)) (justify right bottom))
   )
-  (global_label "USB 5V" (shape input) (at 87.63 43.18 0) (fields_autoplaced)
-    (effects (font (size 1.27 1.27)) (justify left))
-    (property "Intersheetrefs" "${INTERSHEET_REFS}" (at 97.4059 43.18 0)
-      (effects (font (size 1.27 1.27)) (justify left) hide)
-    )
-  )
-  (global_label "DigitalSensorSDA" (shape input) (at 88.265 155.575 0) (fields_autoplaced)
-    (effects (font (size 1.27 1.27)) (justify left))
-    (property "Intersheetrefs" "${INTERSHEET_REFS}" (at 107.3178 155.575 0)
-      (effects (font (size 1.27 1.27)) (justify left) hide)
-    )
-  )
-  (global_label "AnalogueSensorOut" (shape input) (at 88.265 162.56 0) (fields_autoplaced)
-    (effects (font (size 1.27 1.27)) (justify left))
-    (property "Intersheetrefs" "${INTERSHEET_REFS}" (at 109.3738 162.56 0)
-      (effects (font (size 1.27 1.27)) (justify left) hide)
-    )
+  (label "DigitalSensorSDA" (at 88.265 155.575 0) (fields_autoplaced)
+    (effects (font (size 1.27 1.27)) (justify left bottom))
   )
   (sheet (at 16.51 15.24) (size 71.12 87.63) (fields_autoplaced)
@@
       (effects (font (size 1.27 1.27)) (justify right))
     )
-    (pin "AnalogueSensorOut" input (at 88.265 162.56 0)
-      (effects (font (size 1.27 1.27)) (justify right))
-    )
     (instances
       (project "Main"
@@
       (effects (font (size 1.27 1.27)) (justify left))
     )
-    (pin "AnalogueSensorOut" input (at 219.075 76.2 180)
-      (effects (font (size 1.27 1.27)) (justify left))
-    )

Commit message: changes
Other:
- sheet Interfacing ports: added BatterySense; removed none
- sheet Sensing Module ports: added BatterySense; removed none
- title: (none) -> Main Schematic
Changed lines of the file:
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@@
 (kicad_sch (version 20230121) (generator eeschema)
   (paper "A4")
+  (title_block
+    (title "Main Schematic")
+    (date "2023-03-11")
+    (rev "2")
+    (comment 2 "Holly Lewis, Queto Jenkins, Matt Pettit")
+    (comment 3 "Authors: Group 29")
+  )
+  (label "BatterySense" (at 219.075 75.565 180) (fields_autoplaced)
+    (effects (font (size 1.27 1.27)) (justify right bottom))
+  )
   (label "DigitalSensorSCL" (at 88.265 146.685 0) (fields_autoplaced)
     (effects (font (size 1.27 1.27)) (justify left bottom))
@@
   )
   (label "Regulated 3v3" (at 87.63 50.8 0) (fields_autoplaced)
+    (effects (font (size 1.27 1.27)) (justify left bottom))
+  )
+  (label "BatterySense" (at 88.265 160.655 0) (fields_autoplaced)
     (effects (font (size 1.27 1.27)) (justify left bottom))
   )
@@
       (effects (font (size 1.27 1.27)) (justify right))
     )
+    (pin "BatterySense" input (at 88.265 160.655 0)
+      (effects (font (size 1.27 1.27)) (justify right))
+    )
     (instances
       (project "Main"
@@
       (effects (font (size 1.27 1.27)) (justify left))
     )
-    (pin "USB 5V" input (at 219.075 24.765 180)
-      (effects (font (size 1.27 1.27)) (justify left))
-    )
     (pin "DigitalSensorSDA" input (at 219.075 67.31 180)
       (effects (font (size 1.27 1.27)) (justify left))
@@
       (effects (font (size 1.27 1.27)) (justify left))
     )
+    (pin "BatterySense" input (at 219.075 75.565 180)
+      (effects (font (size 1.27 1.27)) (justify left))
+    )
+    (pin "USB 5V" input (at 219.075 24.765 180)
+      (effects (font (size 1.27 1.27)) (justify left))
+    )
