File: Design-files/Main/interfacing.kicad_sch (KiCad schematic)
At the start: 8 parts, among them J1 USB_B_Micro, J3 Conn_01x24_Socket, J4 Conn_01x24_Socket, J5 Conn_01x24_Pin, J6 Conn_01x24_Pin, J7 Conn_01x10_Pin, U1 CH340C, U2 CAT24C256

Commit message: Lots of changes :)
Parts:
- J1: footprint (none) -> Connector_USB:USB_Mini-B_Lumberg_2486_01_Horizontal
- J3: renamed from J5; footprint (none) -> Connector_PinHeader_2.54mm:PinHeader_1x24_P2.54mm_Vertical
- J4: renamed from J3; footprint (none) -> Connector_PinSocket_2.54mm:PinSocket_1x24_P2.54mm_Vertical
- J5: renamed from J4; footprint (none) -> Connector_PinSocket_2.54mm:PinSocket_1x24_P2.54mm_Vertical
- J6: footprint (none) -> Connector_PinHeader_2.54mm:PinHeader_1x24_P2.54mm_Vertical
- J7: footprint (none) -> Connector_PinHeader_2.54mm:PinHeader_1x10_P2.54mm_Vertical
- U1: footprint Package_SO:SOIC-16_3.9x9.9mm_P1.27mm -> Package_SO:SOIC-8W_5.3x5.3mm_P1.27mm
- U2: footprint (none) -> Package_TO_SOT_SMD:SOT-89-3
Connections:
- net USART_RX: now also U1.2 (TXD); no longer U1.3 (RXD)
- net USART_TX: now also U1.3 (RXD); no longer U1.2 (TXD)
- net AnalogueSensorOut renamed Battery
- no-connect marks 3 -> 12
Other:
- note added: "Debug Pins"
- note removed: "10x Debug Pins"
- title: (none) -> Interfacing Schematic

Commit message: changes
Parts:
- added C8, C9: 0.1uF, symbol Device:C
- added J13: Conn_01x02_Pin, symbol Connector:Conn_01x02_Pin
- added R11, R12: 4700, symbol Device:R
- added R13 (x7), R14: 0, symbol Device:R
Connections:
- net 3v3 Regulated: now also R13.1, R13.1; no longer U1.16 (VCC), U2.8 (VCC)
- net EEPROMSCL: now also R14.1; no longer U2.6 (SCL)
- net EEPROMSDA: now also R13.1; no longer U2.5 (SDA)
- net GND: now also C8.2, C9.2
- net USART_RX: now also R13.1; no longer U1.2 (TXD)
- net USART_TX: now also R13.2; no longer U1.3 (RXD)
- net USB D+: now also J13.2 (Pin_2), R13.2; no longer U1.5 (UD+)
- net USB D-: now also J13.1 (Pin_1), R13.2; no longer U1.6 (UD-)
- net at U1.4 (V3): now also C8.1
- net Battery renamed BatterySense
- new net: R12.2, R13.2, U2.5 (SDA)
- new net: R11.2, R14.2, U2.6 (SCL)
- new net: R11.1, R12.1, R13.2, U2.8 (VCC)
- new net: R13.1, U1.6 (UD-)
- new net: C9.1, R13.2, U1.16 (VCC)
- new net: R13.2, U1.2 (TXD)
- new net: R13.1, U1.3 (RXD)
- new net: R13.1, U1.5 (UD+)
- no-connect marks 12 -> 11
Other:
- note added: "Pins Available In case of module failure"
- note added: "Required 10x Debug Pins"
- moved on the sheet: J7, U1, U2

Commit message: changes
Parts:
- C8, C9: footprint (none) -> Capacitor_SMD:C_0201_0603Metric
- J13: footprint (none) -> Connector_PinHeader_2.54mm:PinHeader_1x02_P2.54mm_Vertical
- R11, R12, R13, R14: footprint (none) -> Resistor_SMD:R_0201_0603Metric
Changed lines of the file:
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@@
       (effects (font (size 1.27 1.27)))
     )
-    (property "Footprint" "" (at 50.165 55.118 90)
+    (property "Footprint" "Resistor_SMD:R_0201_0603Metric" (at 50.165 55.118 90)
       (effects (font (size 1.27 1.27)) hide)
     )
@@
       (effects (font (size 1.27 1.27)))
     )
-    (property "Footprint" "" (at 132.842 80.01 90)
+    (property "Footprint" "Resistor_SMD:R_0201_0603Metric" (at 132.842 80.01 90)
       (effects (font (size 1.27 1.27)) hide)
     )
@@
       (effects (font (size 1.27 1.27)))
     )
-    (property "Footprint" "" (at 69.85 32.893 90)
+    (property "Footprint" "Resistor_SMD:R_0201_0603Metric" (at 69.85 32.893 90)
       (effects (font (size 1.27 1.27)) hide)
     )
@@
       (effects (font (size 1.27 1.27)))
     )
-    (property "Footprint" "" (at 130.302 80.01 90)
+    (property "Footprint" "Resistor_SMD:R_0201_0603Metric" (at 130.302 80.01 90)
       (effects (font (size 1.27 1.27)) hide)
     )
@@
       (effects (font (size 1.27 1.27)) (justify left))
     )
-    (property "Footprint" "" (at 140.335 65.278 90)
+    (property "Footprint" "Resistor_SMD:R_0201_0603Metric" (at 140.335 65.278 90)
       (effects (font (size 1.27 1.27)) hide)
     )
@@
       (effects (font (size 1.27 1.27)) (justify right))
     )
-    (property "Footprint" "" (at 133.35 177.8 0)
+    (property "Footprint" "Connector_PinHeader_2.54mm:PinHeader_1x02_P2.54mm_Vertical" (at 133.35 177.8 0)
       (effects (font (size 1.27 1.27)) hide)
     )
@@
       (effects (font (size 1.27 1.27)))
     )
-    (property "Footprint" "" (at 50.165 32.0802 0)
+    (property "Footprint" "Capacitor_SMD:C_0201_0603Metric" (at 50.165 32.0802 0)
       (effects (font (size 1.27 1.27)) hide)
     )
@@
       (effects (font (size 1.27 1.27)))
     )
-    (property "Footprint" "" (at 149.225 49.403 90)
+    (property "Footprint" "Resistor_SMD:R_0201_0603Metric" (at 149.225 49.403 90)
       (effects (font (size 1.27 1.27)) hide)
     )
@@
       (effects (font (size 1.27 1.27)) (justify left))
     )
-    (property "Footprint" "" (at 140.335 72.263 90)
+    (property "Footprint" "Resistor_SMD:R_0201_0603Metric" (at 140.335 72.263 90)
       (effects (font (size 1.27 1.27)) hide)
     )
@@
       (effects (font (size 1.27 1.27)))
     )
-    (property "Footprint" "" (at 50.165 38.4302 0)
+    (property "Footprint" "Capacitor_SMD:C_0201_0603Metric" (at 50.165 38.4302 0)
       (effects (font (size 1.27 1.27)) hide)
     )
@@
       (effects (font (size 1.27 1.27)))
     )
-    (property "Footprint" "" (at 80.645 44.958 90)
+    (property "Footprint" "Resistor_SMD:R_0201_0603Metric" (at 80.645 44.958 90)
       (effects (font (size 1.27 1.27)) hide)
     )
@@
       (effects (font (size 1.27 1.27)))
     )
-    (property "Footprint" "" (at 50.165 52.578 90)
+    (property "Footprint" "Resistor_SMD:R_0201_0603Metric" (at 50.165 52.578 90)
       (effects (font (size 1.27 1.27)) hide)
     )
@@
       (effects (font (size 1.27 1.27)))
     )
-    (property "Footprint" "" (at 80.645 43.942 90)
-      (effects (font (size 1.27 1.27)) hide)
-    )
+    (property "Footprint" "Resistor_SMD:R_0201_0603Metric" (at 80.645 43.942 90)
+      (effects (font (size 1.27 1.27)) hide)
+    )

Commit message: lets go team
Parts:
- R11, R12: value 4700 -> 4.7k
- renumbered J3 to J3-Left1, J4 to J4-Left1, J5 to J5-Right1, J6 to J6-Right1
Other:
- moved on the sheet: J1, J3-Left1, J4-Left1, J5-Right1, J6-Right1

Commit message: lots of changes
Parts:
- removed C8, C9: 0.1uF, Capacitor_SMD:C_0201_0603Metric, symbol Device:C
- removed R13 (x6): 0, Resistor_SMD:R_0201_0603Metric, symbol Device:R
- removed U1: CH340C, Package_SO:SOIC-8W_5.3x5.3mm_P1.27mm, symbol Interface_USB:CH340C
- removed U2: CAT24C256, Package_TO_SOT_SMD:SOT-89-3, symbol Memory_EEPROM:CAT24C256
- added C5, C6: 0.1uF, footprint:C1206, symbol Device:C
- added R13 (x6): 0, footprint:R0402, symbol Device:R
- added U1: CH340C, footprint:SOP-16_L10.0-W3.9-P1.27-LS6.0-BL, symbol CH340C:CH340C
- added U7: M24C64-RMN6TP, footprint:SOIC-8_L5.0-W4.0-P1.27-LS6.0-BL, symbol M24C64-RMN6TP:M24C64-RMN6TP
- R11, R12, R13, R14: footprint Resistor_SMD:R_0201_0603Metric -> footprint:R0402
Connections:
- net 3v3 Regulated: now also R13.1, R13.1
- net GND: now also C5.2, C6.2, U1.1 (GND), U7.1 (A0), U7.2 (A1), U7.3 (A2), U7.4 (VSS)
- net USART_RX: now also R13.2
- net USART_TX: now also R13.2
- net USB D+: now also R13.2
- net USB D-: now also R13.2
- net at R12.2, R13.2: now also U7.6 (SCL)
- net at R11.2, R14.2: now also U7.5 (SDA)
- net at R11.1, R12.1: now also R13.2, U7.8 (VCC)
- new net: R13.1, U1.5 (D+)
- new net: C6.1, R13.2, U1.16 (VCC)
- new net: R13.1, U1.2 (TXD)
- new net: R13.1, U1.3 (RXD)
- new net: C5.1, U1.4 (V3)
- new net: R13.1, U1.6 (D-)
- no-connect marks 11 -> 14
Other:
- moved on the sheet: J1, R11, R12, R13, R14
