File: Design-files/Main/Main.kicad_pcb (KiCad board)
At the start: 2 copper layers, 99.5 x 90.4 mm, 57 parts, among them J1 USB_B_Micro, J13 Conn_01x02_Pin, J2 Battery Jumper, J3-Left1 Conn_01x24_Pin, J4-Left1 Conn_01x24_Socket, J5-Right1 Conn_01x24_Socket, J6-Right1 Conn_01x24_Pin, J7 Conn_01x10_Pin, J8 Conn_01x04_Pin, J9 Conn_01x02_Pin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

Commit message: gerbiees and silkscrenno
Other:
- board text added: "EEE3088F 2023"
- board text added: "GROUP TEN"
- board text added: "JNKKET001"
- board text added: "LWSHOL001"
- board text added: "PTTMAT005"
- board text added: "PWR DEBUG PINS"
- board text added: "SENSOR DEBUG PINS"
- board text added: "V 04"
- board text removed: "DEBUG PINS"
Changed lines of the file:
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@@
     (property "ki_keywords" "cap capacitor")
     (attr through_hole)
-    (fp_text reference "C3" (at 0 -2.68 90) (layer "F.SilkS")
+    (fp_text reference "C3" (at -3.592583 -0.05 -180) (layer "F.SilkS")
         (effects (font (size 1 1) (thickness 0.15)))
     )
@@
     (property "ki_keywords" "R res resistor")
     (attr through_hole)
-    (fp_text reference "R9" (at 0.91 1.789) (layer "F.SilkS")
+    (fp_text reference "R9" (at -2.19 -0.111) (layer "F.SilkS")
         (effects (font (size 1 1) (thickness 0.15)))
     )
@@
     (fp_arc (start 1.080188 -0.709627) (mid 1.299286 -0.618875) (end 1.390018 -0.399772)
       (stroke (width 0.254) (type solid)) (layer "F.SilkS"))
-    (fp_arc (start 1.390018 0.400203) (mid 1.299267 0.619284) (end 1.080188 0.710033)
+    (fp_arc (start 1.390018 0.400203) (mid 1.299267 0.61928) (end 1.080188 0.710033)
       (stroke (width 0.254) (type solid)) (layer "F.SilkS"))
     (fp_circle (center -0.800102 0.400051) (end -0.77013 0.400051)
@@
     (property "ki_keywords" "R res resistor")
     (attr through_hole)
-    (fp_text reference "R23" (at 0 1.756 90) (layer "F.SilkS")
+    (fp_text reference "R23" (at 0 -1.496 90) (layer "F.SilkS")
         (effects (font (size 1 1) (thickness 0.15)))
     )
@@
     (property "ki_keywords" "R res resistor")
     (attr through_hole)
-    (fp_text reference "R28" (at 0.152817 1.776 180) (layer "F.SilkS")
+    (fp_text reference "R28" (at 0.092817 -1.704 180) (layer "F.SilkS")
         (effects (font (size 1 1) (thickness 0.15)))
     )
@@
     (property "ki_keywords" "R res resistor")
     (attr through_hole)
-    (fp_text reference "R10" (at 2.060817 -0.072 90) (layer "F.SilkS")
+    (fp_text reference "R10" (at 0 -1.4 180) (layer "F.SilkS")
         (effects (font (size 1 1) (thickness 0.15)))
     )
@@
     (fp_arc (start 1.080188 -0.709627) (mid 1.299286 -0.618875) (end 1.390018 -0.399772)
       (stroke (width 0.254) (type solid)) (layer "F.SilkS"))
-    (fp_arc (start 1.390018 0.400203) (mid 1.299267 0.619284) (end 1.080188 0.710033)
+    (fp_arc (start 1.390018 0.400203) (mid 1.299267 0.61928) (end 1.080188 0.710033)
       (stroke (width 0.254) (type solid)) (layer "F.SilkS"))
     (fp_circle (center -0.800102 0.400051) (end -0.77013 0.400051)
@@
     (property "ki_keywords" "connector")
     (attr through_hole)
-    (fp_text reference "J3-Left1" (at 5 -0.36) (layer "F.SilkS") hide
+    (fp_text reference "J3-Left1" (at 0.2 -2.36) (layer "F.SilkS")
         (effects (font (size 1 1) (thickness 0.15)))
     )
@@
     (property "ki_keywords" "connector")
     (attr through_hole)
-    (fp_text reference "J6-Right1" (at -2.8 -2.14) (layer "F.SilkS")
+    (fp_text reference "J6-Right1" (at 0 -2.54) (layer "F.SilkS")
         (effects (font (size 1 1) (thickness 0.15)))
     )
@@
     (property "ki_keywords" "connector")
     (attr through_hole)
-    (fp_text reference "J2" (at 1.33 3.87) (layer "F.SilkS")
+    (fp_text reference "J2" (at 2.532 2.584) (layer "F.SilkS")
         (effects (font (size 1 1) (thickness 0.15)))
     )
@@
     (property "ki_keywords" "connector")
     (attr through_hole)
-    (fp_text reference "J9" (at -3.048 1.016 180) (layer "F.SilkS")
+    (fp_text reference "J9" (at 0.088 -3.232 180) (layer "F.SilkS")
         (effects (font (size 1 1) (thickness 0.15)))
     )
@@
     (property "ki_keywords" "R res resistor")
     (attr smd)
-    (fp_text reference "R2" (at 1.584 0.16 180) (layer "F.SilkS")
+    (fp_text reference "R2" (at 0.061 1.36 180) (layer "F.SilkS")
         (effects (font (size 1 1) (thickness 0.15)))
     )
@@
     (property "ki_keywords" "R res resistor")
     (attr through_hole)
-    (fp_text reference "R8" (at 2.432817 0.05) (layer "F.SilkS")
+    (fp_text reference "R8" (at 0.032817 -1.55) (layer "F.SilkS")
         (effects (font (size 1 1) (thickness 0.15)))
     )
@@
     (property "ki_keywords" "connector")
     (attr through_hole)
-    (fp_text reference "J4-Left1" (at 0 -2.77) (layer "F.SilkS")
+    (fp_text reference "J4-Left1" (at -0.02 -2.77) (layer "F.SilkS")
         (effects (font (size 1 1) (thickness 0.15)))
     )
@@
     (property "ki_keywords" "R res resistor")
     (attr through_hole)
-    (fp_text reference "R6" (at 1.980817 -0.036 90) (layer "F.SilkS")
+    (fp_text reference "R6" (at -0.055183 1.556 180) (layer "F.SilkS")
         (effects (font (size 1 1) (thickness 0.15)))
     )
@@
     (property "ki_keywords" "R res resistor")
     (attr smd)
-    (fp_text reference "R3" (at 0.003 -2.308) (layer "F.SilkS")
+    (fp_text reference "R3" (at -1.824 0.04) (layer "F.SilkS")
         (effects (font (size 1 1) (thickness 0.15)))
     )
@@
     (property "ki_keywords" "connector")
     (attr through_hole)
-    (fp_text reference "J5-Right1" (at -1.4 -1.14) (layer "F.SilkS")
+    (fp_text reference "J5-Right1" (at 0 -2.54) (layer "F.SilkS")
         (effects (font (size 1 1) (thickness 0.15)))
     )
@@
     (property "ki_keywords" "R res resistor")
     (attr through_hole)
-    (fp_text reference "R16" (at 2.703 0) (layer "F.SilkS")
+    (fp_text reference "R16" (at 0.05 -1.4) (layer "F.SilkS")
         (effects (font (size 1 1) (thickness 0.15)))
     )
@@
     (property "ki_keywords" "diode Schottky")
     (attr through_hole)
-    (fp_text reference "D1" (at 4.134595 -2.05 180) (layer "F.SilkS")
+    (fp_text reference "D1" (at 0.215405 -0.05 180) (layer "F.SilkS")
         (effects (font (size 1 1) (thickness 0.15)))
     )
@@
     )
   )
-  (gr_rect (start 116.79 47.58081) (end 121.5 62.84081)
+  (gr_rect (start 116.79 47.58081) (end 121.5 63.8)
     (stroke (width 0.1) (type default)) (fill none) (layer "F.SilkS"))
   (gr_rect (start 152.8 46.6) (end 171.6 65.8)
     (stroke (width 0.1) (type default)) (fill none) (layer "F.SilkS"))
-  (gr_rect (start 174.05 51.95) (end 185.45 62.55)
+  (gr_rect (start 174.05 51.95) (end 185.6 65.8)
     (stroke (width 0.1) (type default)) (fill none) (layer "F.SilkS"))
   (gr_line (start 165.546 110.883) (end 180.946 110.883)
     (stroke (width 0.1) (type default)) (layer "F.SilkS"))
+  (gr_rect (start 135.6 71.4) (end 148.8 101.2)
+    (stroke (width 0.1) (type default)) (fill none) (layer "F.SilkS"))
   (gr_line (start 165.546 130.683) (end 165.546 110.883)
     (stroke (width 0.1) (type default)) (layer "F.SilkS"))
@@
   (gr_line (start 192.532 135.382) (end 93.0148 135.382)
     (stroke (width 0.05) (type default)) (layer "Edge.Cuts"))
+  (gr_text "GROUP TEN" (at 137.4 80.2) (layer "F.SilkS")
+    (effects (font (size 1 1) (thickness 0.1)) (justify left bottom))
+  )
+  (gr_text "EEE3088F 2023" (at 136.2 74.8) (layer "F.SilkS")
+    (effects (font (size 1 1) (thickness 0.1)) (justify left bottom))
+  )
   (gr_text "FTDI\nMODULE" (at 187.146 131.283 90) (layer "F.SilkS")
     (effects (font (size 1 1) (thickness 0.1)) (justify left bottom))
@@
     (effects (font (size 1 1) (thickness 0.1)) (justify left bottom))
   )
-  (gr_text "VOLTAGE\nREGULATOR" (at 173.35 65.4) (layer "F.SilkS")
+  (gr_text "JNKKET001" (at 137.4 86.2) (layer "F.SilkS")
+    (effects (font (size 1 1) (thickness 0.1)) (justify left bottom))
+  )
+  (gr_text "VOLTAGE\nREGULATOR" (at 174.05 65.8) (layer "F.SilkS")
     (effects (font (size 0.9 1) (thickness 0.09)) (justify left bottom))
   )
+  (gr_text "V 04" (at 144.8 100.8) (layer "F.SilkS")
+    (effects (font (size 1 1) (thickness 0.1)) (justify left bottom))
+  )
+  (gr_text "PWR DEBUG PINS\n" (at 174 47.4) (layer "F.SilkS")
+    (effects (font (size 1 1) (thickness 0.1)) (justify left bottom))
+  )
   (gr_text "PWR SWITCHING CCT" (at 154.95 64.9) (layer "F.SilkS")
     (effects (font (size 1 1) (thickness 0.1)) (justify left bottom))
   )
+  (gr_text "PTTMAT005\n" (at 137.6 84.4) (layer "F.SilkS")
+    (effects (font (size 1 1) (thickness 0.1)) (justify left bottom))
+  )
   (gr_text "TEMPERATURE AND HUMIDITY\nDIGITAL SENSOR" (at 177.29 91.836 90) (layer "F.SilkS")
     (effects (font (size 1 1) (thickness 0.1)) (justify left bottom))
   )
-  (gr_text "DEBUG\nPINS" (at 168.656 100.584) (layer "F.SilkS")
+  (gr_text "SENSOR DEBUG PINS" (at 172.4 83 90) (layer "F.SilkS")
     (effects (font (size 1 1) (thickness 0.1)) (justify bottom))
   )
-  (gr_text "Battery Connect\n" (at 118.25 62.43081 90) (layer "F.SilkS")
+  (gr_text "LWSHOL001" (at 137.4 82.4) (layer "F.SilkS")
+    (effects (font (size 1 1) (thickness 0.1)) (justify left bottom))
+  )
+  (gr_text "Battery Connect\n" (at 118 63.6 90) (layer "F.SilkS")
     (effects (font (size 1 1) (thickness 0.1)) (justify left bottom))
   )
